File: AT90S4433_evaluation_board/AT90S4433_evaluation_board.kicad_sch (KiCad schematic)
At the start: 25 parts, among them SW1 USR_BTN, Y1 Crystal_Small

Commit message: corrections
Parts:
- added R5: R, Resistor_SMD:R_0805_2012Metric, symbol Device:R
- D3: footprint Diode_THT:D_DO-41_SOD81_P10.16mm_Horizontal -> Diode_SMD:D_2512_6332Metric
Connections:
- net VCC: now also R5.2; no longer D3.1 (K)
- new net: D3.1 (K), R5.1
Other:
- moved on the sheet: R4
Changed lines of the file:
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@@
   (junction (at 47.625 77.47) (diameter 0) (color 0 0 0 0)
   )
+  (junction (at 190.5 120.65) (diameter 0) (color 0 0 0 0)
+  )
   (junction (at 92.075 49.53) (diameter 0) (color 0 0 0 0)
   )
@@
   (junction (at 100.965 49.53) (diameter 0) (color 0 0 0 0)
   )
-  (junction (at 190.5 125.095) (diameter 0) (color 0 0 0 0)
-  )
-  (junction (at 172.085 125.095) (diameter 0) (color 0 0 0 0)
-  )
   (junction (at 165.1 44.45) (diameter 0) (color 0 0 0 0)
   )
@@
   )
   (junction (at 34.925 71.755) (diameter 0) (color 0 0 0 0)
+  )
+  (junction (at 172.085 120.65) (diameter 0) (color 0 0 0 0)
   )
   (junction (at 47.625 65.405) (diameter 0) (color 0 0 0 0)
@@
     (stroke (width 0) (type default))
   )
-  (wire (pts (xy 172.085 125.095) (xy 172.085 128.27))
-    (stroke (width 0) (type default))
-  )
   (wire (pts (xy 100.965 49.53) (xy 125.73 49.53))
     (stroke (width 0) (type default))
@@
     (stroke (width 0) (type default))
   )
+  (wire (pts (xy 205.74 120.65) (xy 205.74 125.095))
+    (stroke (width 0) (type default))
+  )
   (wire (pts (xy 146.05 66.04) (xy 149.86 66.04))
     (stroke (width 0) (type default))
@@
     (stroke (width 0) (type default))
   )
-  (wire (pts (xy 26.035 145.415) (xy 26.035 144.145))
+  (wire (pts (xy 26.035 146.05) (xy 26.035 144.78))
     (stroke (width 0) (type default))
   )
@@
     (stroke (width 0) (type default))
   )
+  (wire (pts (xy 190.5 120.65) (xy 205.74 120.65))
+    (stroke (width 0) (type default))
+  )
   (wire (pts (xy 172.085 136.525) (xy 172.085 135.89))
     (stroke (width 0) (type default))
@@
     (stroke (width 0) (type default))
   )
+  (wire (pts (xy 26.035 137.16) (xy 26.035 136.525))
+    (stroke (width 0) (type default))
+  )
   (wire (pts (xy 120.015 63.5) (xy 125.73 63.5))
     (stroke (width 0) (type default))
@@
     (stroke (width 0) (type default))
   )
+  (wire (pts (xy 172.085 120.65) (xy 172.085 128.27))
+    (stroke (width 0) (type default))
+  )
   (wire (pts (xy 120.015 78.74) (xy 125.73 78.74))
     (stroke (width 0) (type default))
   )
-  (wire (pts (xy 172.085 125.095) (xy 190.5 125.095))
-    (stroke (width 0) (type default))
-  )
   (wire (pts (xy 120.015 73.66) (xy 125.73 73.66))
     (stroke (width 0) (type default))
@@
     (stroke (width 0) (type default))
   )
-  (wire (pts (xy 172.085 124.46) (xy 172.085 125.095))
-    (stroke (width 0) (type default))
-  )
   (wire (pts (xy 165.1 36.195) (xy 165.1 36.83))
     (stroke (width 0) (type default))
   )
-  (wire (pts (xy 190.5 125.095) (xy 205.74 125.095))
-    (stroke (width 0) (type default))
-  )
   (wire (pts (xy 205.74 135.255) (xy 205.74 135.89))
     (stroke (width 0) (type default))
@@
     (stroke (width 0) (type default))
   )
-  (wire (pts (xy 190.5 125.095) (xy 190.5 128.27))
-    (stroke (width 0) (type default))
-  )
   (wire (pts (xy 146.05 63.5) (xy 149.86 63.5))
     (stroke (width 0) (type default))
   )
+  (wire (pts (xy 26.035 127) (xy 26.035 128.905))
+    (stroke (width 0) (type default))
+  )
   (wire (pts (xy 28.575 71.755) (xy 28.575 72.39))
     (stroke (width 0) (type default))
@@
     (stroke (width 0) (type default))
   )
+  (wire (pts (xy 172.085 120.65) (xy 190.5 120.65))
+    (stroke (width 0) (type default))
+  )
   (wire (pts (xy 47.625 73.66) (xy 47.625 77.47))
     (stroke (width 0) (type default))
@@
     (effects (font (size 1.27 1.27)) (justify left bottom))
   )
-  (text "Simple power supply and protection\n" (at 159.385 116.205 0)
+  (text "Simple power supply and protection\n" (at 169.545 110.49 0)
     (effects (font (size 1.27 1.27)) (justify left bottom))
   )
@@
     )
   )
-  (symbol (lib_id "power:VCC") (at 26.035 128.905 0) (unit 1)
-    (in_bom yes) (on_board yes) (dnp no) (fields_autoplaced)
-    (property "Reference" "#PWR013" (at 26.035 132.715 0)
-      (effects (font (size 1.27 1.27)) hide)
-    )
-    (property "Value" "VCC" (at 26.035 123.825 0)
-      (effects (font (size 1.27 1.27)))
-    )
-    (property "Footprint" "" (at 26.035 128.905 0)
-      (effects (font (size 1.27 1.27)) hide)
-    )
-    (property "Datasheet" "" (at 26.035 128.905 0)
+  (symbol (lib_id "power:VCC") (at 26.035 127 0) (unit 1)
+    (in_bom yes) (on_board yes) (dnp no) (fields_autoplaced)
+    (property "Reference" "#PWR013" (at 26.035 130.81 0)
+      (effects (font (size 1.27 1.27)) hide)
+    )
+    (property "Value" "VCC" (at 26.035 121.92 0)
+      (effects (font (size 1.27 1.27)))
+    )
+    (property "Footprint" "" (at 26.035 127 0)
+      (effects (font (size 1.27 1.27)) hide)
+    )
+    (property "Datasheet" "" (at 26.035 127 0)
       (effects (font (size 1.27 1.27)) hide)
     )
@@
     )
   )
-  (symbol (lib_id "power:GND") (at 26.035 145.415 0) (unit 1)
-    (in_bom yes) (on_board yes) (dnp no) (fields_autoplaced)
-    (property "Reference" "#PWR08" (at 26.035 151.765 0)
-      (effects (font (size 1.27 1.27)) hide)
-    )
-    (property "Value" "GND" (at 26.035 150.495 0)
-      (effects (font (size 1.27 1.27)))
-    )
-    (property "Footprint" "" (at 26.035 145.415 0)
-      (effects (font (size 1.27 1.27)) hide)
-    )
-    (property "Datasheet" "" (at 26.035 145.415 0)
+  (symbol (lib_id "power:GND") (at 26.035 146.05 0) (unit 1)
+    (in_bom yes) (on_board yes) (dnp no) (fields_autoplaced)
+    (property "Reference" "#PWR08" (at 26.035 152.4 0)
+      (effects (font (size 1.27 1.27)) hide)
+    )
+    (property "Value" "GND" (at 26.035 151.13 0)
+      (effects (font (size 1.27 1.27)))
+    )
+    (property "Footprint" "" (at 26.035 146.05 0)
+      (effects (font (size 1.27 1.27)) hide)
+    )
+    (property "Datasheet" "" (at 26.035 146.05 0)
       (effects (font (size 1.27 1.27)) hide)
     )
@@
     )
   )
-  (symbol (lib_id "power:VCC") (at 172.085 124.46 0) (unit 1)
-    (in_bom yes) (on_board yes) (dnp no) (fields_autoplaced)
-    (property "Reference" "#PWR010" (at 172.085 128.27 0)
-      (effects (font (size 1.27 1.27)) hide)
-    )
-    (property "Value" "VCC" (at 172.085 119.38 0)
-      (effects (font (size 1.27 1.27)))
-    )
-    (property "Footprint" "" (at 172.085 124.46 0)
-      (effects (font (size 1.27 1.27)) hide)
-    )
-    (property "Datasheet" "" (at 172.085 124.46 0)
+  (symbol (lib_id "power:VCC") (at 172.085 120.65 0) (unit 1)
+    (in_bom yes) (on_board yes) (dnp no) (fields_autoplaced)
+    (property "Reference" "#PWR010" (at 172.085 124.46 0)
+      (effects (font (size 1.27 1.27)) hide)
+    )
+    (property "Value" "VCC" (at 172.085 115.57 0)
+      (effects (font (size 1.27 1.27)))
+    )
+    (property "Footprint" "" (at 172.085 120.65 0)
+      (effects (font (size 1.27 1.27)) hide)
+    )
+    (property "Datasheet" "" (at 172.085 120.65 0)
       (effects (font (size 1.27 1.27)) hide)
     )
@@
     )
   )
+  (symbol (lib_id "Device:R") (at 190.5 124.46 180) (unit 1)
+    (in_bom yes) (on_board yes) (dnp no) (fields_autoplaced)
+    (property "Reference" "R5" (at 193.04 123.19 0)
+      (effects (font (size 1.27 1.27)) (justify right))
+    )
+    (property "Value" "R" (at 193.04 125.73 0)
+      (effects (font (size 1.27 1.27)) (justify right))
+    )
+    (property "Footprint" "Resistor_SMD:R_0805_2012Metric" (at 192.278 124.46 90)
+      (effects (font (size 1.27 1.27)) hide)
+    )
+    (property "Datasheet" "~" (at 190.5 124.46 0)
+      (effects (font (size 1.27 1.27)) hide)
+    )
+    (pin "1")
+    (pin "2")
+    (instances
+      (project "AT90S4433_evaluation_board"
+        (path "/7ff8dc4c-cb91-450f-a04d-1629054ff54a"
+          (reference "R5") (unit 1)
+        )
+      )
+    )
+  )
   (symbol (lib_id "Device:C") (at 100.965 53.34 180) (unit 1)
     (in_bom yes) (on_board yes) (dnp no) (fields_autoplaced)
@@
     )
   )
-  (symbol (lib_id "Device:R") (at 26.035 140.335 180) (unit 1)
-    (in_bom yes) (on_board yes) (dnp no) (fields_autoplaced)
-    (property "Reference" "R4" (at 28.575 139.065 0)
-      (effects (font (size 1.27 1.27)) (justify right))
-    )
-    (property "Value" "R" (at 28.575 141.605 0)
-      (effects (font (size 1.27 1.27)) (justify right))
-    )
-    (property "Footprint" "Resistor_SMD:R_0805_2012Metric" (at 27.813 140.335 90)
-      (effects (font (size 1.27 1.27)) hide)
-    )
-    (property "Datasheet" "~" (at 26.035 140.335 0)
+  (symbol (lib_id "Device:R") (at 26.035 140.97 180) (unit 1)
+    (in_bom yes) (on_board yes) (dnp no) (fields_autoplaced)
+    (property "Reference" "R4" (at 28.575 139.7 0)
+      (effects (font (size 1.27 1.27)) (justify right))
+    )
+    (property "Value" "R" (at 28.575 142.24 0)
+      (effects (font (size 1.27 1.27)) (justify right))
+    )
+    (property "Footprint" "Resistor_SMD:R_0805_2012Metric" (at 27.813 140.97 90)
+      (effects (font (size 1.27 1.27)) hide)
+    )
+    (property "Datasheet" "~" (at 26.035 140.97 0)
       (effects (font (size 1.27 1.27)) hide)
     )
@@
       (effects (font (size 1.27 1.27)) (justify left))
     )
-    (property "Footprint" "Diode_THT:D_DO-41_SOD81_P10.16mm_Horizontal" (at 190.5 132.08 0)
-      (effects (font (size 1.27 1.27)) hide)
-    )
+    (property "Footprint" "Diode_SMD:D_2512_6332Metric" (at 190.5 132.08 0)
+      (effects (font (size 1.27 1.27)) hide)
+    )

Commit message: footprint name changes, vias corrections, description
Parts:
- JP9: footprint project_lib_footprints:3_pin_jumper_socker -> project_lib_footprints:3_pin_jumper_socket
- TP3: footprint project_lib_footprints:Power_socker -> project_lib_footprints:Power_socket
Changed lines of the file:
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@@
       (effects (font (size 1.27 1.27)) (justify left))
     )
-    (property "Footprint" "project_lib_footprints:3_pin_jumper_socker" (at 170.18 73.66 0)
+    (property "Footprint" "project_lib_footprints:3_pin_jumper_socket" (at 170.18 73.66 0)
       (effects (font (size 1.27 1.27)) hide)
     )
@@
       (effects (font (size 1.27 1.27)) (justify right))
     )
-    (property "Footprint" "project_lib_footprints:Power_socker" (at 205.74 130.175 0)
-      (effects (font (size 1.27 1.27)) hide)
-    )
+    (property "Footprint" "project_lib_footprints:Power_socket" (at 205.74 130.175 0)
+      (effects (font (size 1.27 1.27)) hide)
+    )
